File: PartRight/PartRight.kicad_sch (KiCad schematic)
At the start: 20 parts, among them J1 Left, J2 Middle, J3 LCD, SW1 SW_Push, SW2 SW_Push, SW3 SW_Push, SW4 SW_Push, SW5 SW_Push, SW6 SW_Push, SW7 SW_Push, SW8 SW_Push

Commit message: Fix some rule checks.
Connections:
- no-connect marks 0 -> 10
Changed lines of the file:
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@@
 	(generator_version "9.0")
 	(paper "A4")
+	(no_connect
+		(at 127 74.93)
+	)
+	(no_connect
+		(at 127 67.31)
+	)
+	(no_connect
+		(at 127 54.61)
+	)
+	(no_connect
+		(at 127 52.07)
+	)
+	(no_connect
+		(at 144.78 36.83)
+	)
+	(no_connect
+		(at 127 64.77)
+	)
+	(no_connect
+		(at 127 69.85)
+	)
+	(no_connect
+		(at 172.72 82.55)
+	)
+	(no_connect
+		(at 127 72.39)
+	)
+	(no_connect
+		(at 149.86 36.83)
+	)
 	(global_label "SW3"
 		(shape passive)
